Commit message: real robot arm control

File: dofbot_moveit/urdf/dofbot.urdf (robot description, URDF)
Before this commit: robot yahboom_dofbot, 12 links, 11 joints
Joints:
- joint arm_joint1: axis 0 0 -1 -> 0 0 1
- joint arm_joint2: axis 0 0 -1 -> 0 0 1
- joint arm_joint3: axis 0 0 -1 -> 0 0 1
- joint arm_joint4: axis 0 0 -1 -> 0 0 1
